Commit message: svtrp

File: robot_description/urdf/gazebo_essentials.xacro (robot description, xacro)
@@ -169,6 +169,6 @@
         <plugin name="laser" filename="libgazebo_ros_ray_sensor.so">
           <ros>
-            <namespace>/base</namespace>
-            <remapping>~/out:=laser_scan</remapping>
+            <namespace></namespace>
+            <remapping>~/out:=scan</remapping>
           </ros>
           <output_type>sensor_msgs/LaserScan</output_type>

File: robot_description/urdf/robot_base.xacro (robot description, xacro)
@@ -30,4 +30,12 @@
     </visual>
   </link>
+  <!-- Base FootPrint Link-->
+ <joint name="base_footprint_joint" type="fixed">
+    <origin xyz="0 0 0" rpy="0 0 0" />
+    <parent link="base_link" />
+    <child link="base_footprint" />
+ </joint>
+  <link name="base_footprint">
+  </link>
 <xacro:robot_wheel prefix="front_left" origin="0 0 0"/>
 <xacro:robot_wheel prefix="front_right" origin="0 0 0"/>

Commit message: Nav2 features

File: robot_description/urdf/gazebo_essentials.xacro (robot description, xacro)
@@ -222,3 +222,43 @@
       </sensor>
   </gazebo>
+    <!-- IMU SENSOR -->
+    <gazebo reference="base_IMU_link">
+    <gravity>true</gravity>
+    <sensor name="imu_sensor" type="imu">
+      <always_on>true</always_on>
+      <update_rate>100</update_rate>
+      <visualize>true</visualize>
+      <topic>__default_topic__</topic>
+      <plugin filename="libgazebo_ros_imu_sensor.so" name="imu_plugin">
+        <topicName>imu</topicName>
+        <bodyName>base_IMU_link</bodyName>
+        <updateRateHZ>10.0</updateRateHZ>
+        <gaussianNoise>0.0</gaussianNoise>
+        <xyzOffset>0 0 0</xyzOffset>
+        <rpyOffset>0 0 0</rpyOffset>
+        <frameName>ibase_IMU_link</frameName>
+        <initialOrientationAsReference>false</initialOrientationAsReference>
+        <ros>
+            <namespace></namespace>
+            <remapping>~/out:=imu</remapping>
+          </ros>
+      </plugin>
+      <pose>0 0 0 0 0 0</pose>
+    </sensor>
+  </gazebo>
+  <!-- GPS SENSOR -->
+  <gazebo reference="gps_link">
+    <sensor name="gps_sensor" type="gps">
+        <always_on>true</always_on>
+        <update_rate>1.0</update_rate>
+        <plugin name="gps_controller" filename="libgazebo_ros_gps_sensor.so">
+            <ros>
+                <!-- <namespace>/br</namespace> -->
+                <remapping>gps_controller/out:=gps</remapping>
+            </ros>
+            <frame_name>gps_link</frame_name>
+        </plugin>
+    </sensor>
+    <material>Gazebo/Grey</material>
+</gazebo>
 </robot>

File: robot_description/urdf/robot_base.xacro (robot description, xacro)
@@ -8,4 +8,5 @@
 <xacro:include filename="$(find robot_description)/urdf/camera.xacro" />
 <xacro:include filename="$(find robot_description)/urdf/hokuyo.xacro" />
+<xacro:include filename="$(find robot_description)/urdf/IMU.xacro" />
   <!-- BASE_LINK -->
   <link name="base_link">
@@ -58,3 +59,4 @@
 <xacro:robot_camera/>
 <xacro:robot_lidar/>
+<xacro:base_IMU/>
 </robot>
