Commit message: Visual features: Yolo and OpenCV

File: robot_description/urdf/camera.xacro (robot description, xacro)
@@ -124,10 +124,22 @@
   </link>
   <!-- Depth Camera-->
-   <joint name="camera_depth_joint" type="fixed">
-   <origin xyz="0 0 0" rpy="-1.57075 0 -1.57075"/>
-   <child link="camera_depth_link"/>
-    <parent link="front_camera_link"/>
+  <joint name="camera_depth_joint" type="fixed">
+    <parent link="base_link"/>
+    <child link="camera_depth_link"/>
+    <origin xyz="0.21 0.0 0.0" rpy="0.0 0.0 0.0"/>
   </joint>
-   <link name="camera_depth_link"></link>
+  <link name="camera_depth_link">
+    <visual>
+      <geometry>
+        <mesh filename="package://robot_description/meshes/realsense.dae"/>
+      </geometry>
+    </visual>
+  </link>
+  <joint name="depth_camera_optical_joint" type="fixed">
+    <parent link="camera_depth_link"/>
+    <child link="depth_camera_link_optical"/>
+    <origin xyz="0 0 0" rpy="${-pi/2} 0 ${-pi/2}"/>
+  </joint>
+  <link name="depth_camera_link_optical"></link>
   <!-- POINT CLOUND SENSOR -->
   <link name="pointcloud_link">

File: robot_description/urdf/gazebo_essentials.xacro (robot description, xacro)
@@ -103,46 +103,27 @@
     </gazebo>
         <!-- Depth Camera -->
-  <gazebo reference="front_camera_link">
-     <sensor type="depth" name="depth_camera">
-      <always_on>true</always_on>
-      <camera>
-          <horizontal_fov>1.3439</horizontal_fov>
-          <image>
-              <width>1920</width>
-              <height>1080</height>
-              <format>R8G8B8</format>
-          </image>
-          <depth_camera></depth_camera>
-          <clip>
-              <near>0.03</near>
-              <far>8</far>
-          </clip>
-      </camera>
-      <plugin name="intel_realsense_d430_depth_driver" filename="libgazebo_ros_camera.so">
-        <baseline>0.2</baseline>
-        <alwaysOn>true</alwaysOn>
-        <updateRate>30.0</updateRate>
-        <cameraName>depth_camera</cameraName>
-        <frameName>camera_depth_link</frameName>
-        <imageTopicName>rgb/image_raw</imageTopicName>
-        <depthImageTopicName>depth/image_raw</depthImageTopicName>
-        <pointCloudTopicName>depth/points</pointCloudTopicName>
-        <cameraInfoTopicName>rgb/camera_info</cameraInfoTopicName>
-        <depthImageCameraInfoTopicName>depth/camera_info</depthImageCameraInfoTopicName>
-        <pointCloudCutoff>0.4</pointCloudCutoff>
-            <hackBaseline>0.07</hackBaseline>
-            <distortionK1>0.0</distortionK1>
-            <distortionK2>0.0</distortionK2>
-            <distortionK3>0.0</distortionK3>
-            <distortionT1>0.0</distortionT1>
-            <distortionT2>0.0</distortionT2>
-        <CxPrime>0.0</CxPrime>
-        <Cx>0.0</Cx>
-        <Cy>0.0</Cy>
-        <focalLength>0</focalLength>
-        <hackBaseline>0</hackBaseline>
-      </plugin>
-    </sensor>
-  </gazebo>
+    <gazebo reference="camera_depth_link">
+        <material>Gazebo/Red</material>
+        <sensor name="depth_camera" type="depth">
+            <pose> 0 0 0 0 0 0 </pose>
+            <visualize>true</visualize>
+            <update_rate>10</update_rate>
+            <camera>
+                <horizontal_fov>1.089</horizontal_fov>
+                <image>
+                    <format>R8G8B8</format>
+                    <width>640</width>
+                    <height>480</height>
+                </image>
+                <clip>
+                    <near>0.05</near>
+                    <far>8.0</far>
+                </clip>
+            </camera>
+            <plugin name="camera_controller" filename="libgazebo_ros_camera.so">
+                <frame_name>depth_camera_link_optical</frame_name>
+            </plugin>
+        </sensor>
+    </gazebo>
   <!-- hokuyo -->
   <!-- Sensors -->
@@ -234,14 +215,68 @@
         <bodyName>base_IMU_link</bodyName>
         <updateRateHZ>10.0</updateRateHZ>
-        <gaussianNoise>0.0</gaussianNoise>
+        <gaussianNoise>0.0002</gaussianNoise>
         <xyzOffset>0 0 0</xyzOffset>
         <rpyOffset>0 0 0</rpyOffset>
-        <frameName>ibase_IMU_link</frameName>
+        <frameName>base_IMU_link</frameName>
         <initialOrientationAsReference>false</initialOrientationAsReference>
         <ros>
-            <namespace></namespace>
-            <remapping>~/out:=imu</remapping>
-          </ros>
+          <namespace></namespace>
+          <remapping>~/out:=imu</remapping>
+        </ros>
       </plugin>
+      <imu>
+        <angular_velocity>
+          <x>
+            <noise type="gaussian">
+              <mean>0.0</mean>
+              <stddev>2e-4</stddev>
+              <bias_mean>0.0000075</bias_mean>
+              <bias_stddev>0.0000008</bias_stddev>
+            </noise>
+          </x>
+          <y>
+            <noise type="gaussian">
+              <mean>0.0</mean>
+              <stddev>2e-4</stddev>
+              <bias_mean>0.0000075</bias_mean>
+              <bias_stddev>0.0000008</bias_stddev>
+            </noise>
+          </y>
+          <z>
+            <noise type="gaussian">
+              <mean>0.0</mean>
+              <stddev>2e-4</stddev>
+              <bias_mean>0.0000075</bias_mean>
+              <bias_stddev>0.0000008</bias_stddev>
+            </noise>
+          </z>
+        </angular_velocity>
+        <linear_acceleration>
+          <x>
+            <noise type="gaussian">
+              <mean>0.0</mean>
+              <stddev>1.7e-2</stddev>
+              <bias_mean>0.1</bias_mean>
+              <bias_stddev>0.001</bias_stddev>
+            </noise>
+          </x>
+          <y>
+            <noise type="gaussian">
+              <mean>0.0</mean>
+              <stddev>1.7e-2</stddev>
+              <bias_mean>0.1</bias_mean>
+              <bias_stddev>0.001</bias_stddev>
+            </noise>
+          </y>
+          <z>
+            <noise type="gaussian">
+              <mean>0.0</mean>
+              <stddev>1.7e-2</stddev>
+              <bias_mean>0.1</bias_mean>
+              <bias_stddev>0.001</bias_stddev>
+            </noise>
+          </z>
+        </linear_acceleration>
+      </imu>
       <pose>0 0 0 0 0 0</pose>
     </sensor>

File: robot_description/urdf/hokuyo.xacro (robot description, xacro)
@@ -11,13 +11,13 @@
 	<inertial>
 		<mass value="1e-5" />
-			<origin xyz="0 0 0" rpy="0 0 0"/>
-			<inertia ixx="1e-6" ixy="0" ixz="0" iyy="1e-6" iyz="0" izz="1e-6" />
-		</inertial>
-		<visual>
-			<origin xyz="0 0 0" rpy="0 0 0"/>
-			<geometry>
-				<box size="0.05 0.05 0.05"/>
-			</geometry>
-		</visual>
+		<origin xyz="0 0 0" rpy="0 0 0"/>
+		<inertia ixx="1e-6" ixy="0" ixz="0" iyy="1e-6" iyz="0" izz="1e-6" />
+	</inertial>
+	<visual>
+		<origin xyz="0 0 0" rpy="0 0 0"/>
+		<geometry>
+			<mesh filename="package://robot_description/meshes/hokuyo.dae"/>
+		</geometry>
+	</visual>
 </link>
 <joint name="front_hokuyo_joint" type="fixed">

File: robot_description/urdf/robot_base.xacro (robot description, xacro)
@@ -9,4 +9,5 @@
 <xacro:include filename="$(find robot_description)/urdf/hokuyo.xacro" />
 <xacro:include filename="$(find robot_description)/urdf/IMU.xacro" />
+<xacro:property name="black" value="0.0 0.0 0.0 1"/> <!-- RGBA values -->
   <!-- BASE_LINK -->
   <link name="base_link">
@@ -14,5 +15,5 @@
       <origin xyz="0 0 0.0" rpy="0 0 0" />
       <geometry>
-        <!--<mesh filename="package://mobile_manipulator_body/meshes/robot_base.stl"/>-->
+        <!--mesh filename="package://robot_description/meshes/robot_base.stl"/-->
         <box size="0.38 0.203 0.07" />
       </geometry>
@@ -26,12 +27,17 @@
       <origin xyz="0 0 0" rpy="0 0 0" />
       <geometry>
-        <!--<mesh filename="package://mobile_manipulator_body/meshes/robot_base.stl"/>-->
         <box size="0.38 0.203 0.07" />
       </geometry>
+      <material name="wheel_material">
+        <color rgba="0.0 0.0 0.0 1.0"/>
+    </material>
     </visual>
   </link>
+<gazebo reference="base_link">
+  <material>Gazebo/Black</material>
+</gazebo>
   <!-- Base FootPrint Link-->
  <joint name="base_footprint_joint" type="fixed">
-    <origin xyz="0 0 0" rpy="0 0 0" />
+    <origin xyz="0 0 -0.06" rpy="0 0 0" />
     <parent link="base_link" />
     <child link="base_footprint" />

File: robot_description/urdf/robot_essentials.xacro (robot description, xacro)
@@ -1,42 +1,32 @@
 <?xml version="1.0"?>
 <robot xmlns:xacro="http://ros.org/wiki/xacro" name="robot_essentials" >
+<xacro:property name="wheel_color" value="0.0 0.0 0.0 1"/> <!-- RGBA values -->
 <xacro:macro name="robot_wheel" params="prefix origin">
 <link name="${prefix}_wheel">
-<collision>
-      <origin
-        xyz="${origin}"
-        rpy="1.5707963267949 0 0" />
-      <geometry>
-       <cylinder radius="0.06" length="0.04" />
-      </geometry>
-    </collision>
-    <inertial>
-      <origin
-        xyz="-4.1867E-18 0.0068085 -1.65658661799998E-18"
-        rpy="0 0 0" />
-      <mass
-        value="0.378" />
-      <inertia
-        ixx="0.00856502765719703"
-        ixy="1.5074118157338E-19"
-        ixz="-4.78150098725052E-19"
-        iyy="0.013670640432096"
-        iyz="-2.68136447099727E-19"
-        izz="0.00856502765719703" />
-    </inertial>
-       <visual>
-      <origin
-        xyz="${origin}"
-        rpy="1.5707963267949 0 0" />
-      <geometry>
-       <cylinder radius="0.06" length="0.04" />
-      </geometry>
-      <material
-        name="">
-        <color
-          rgba="0.79216 0.81961 0.93333 1" />
-      </material>
-    </visual>
+  <collision>
+    <origin xyz="${origin}" rpy="1.5707963267949 0 0" />
+    <geometry>
+      <cylinder radius="0.06" length="0.04" />
+    </geometry>
+  </collision>
+  <inertial>
+    <origin xyz="-4.1867E-18 0.0068085 -1.65658661799998E-18" rpy="0 0 0" />
+    <mass value="0.378" />
+    <inertia ixx="0.00856502765719703" ixy="1.5074118157338E-19" ixz="-4.78150098725052E-19"
+        iyy="0.013670640432096" iyz="-2.68136447099727E-19" izz="0.00856502765719703" />
+  </inertial>
+  <visual>
+    <origin xyz="${origin}" rpy="1.5707963267949 0 0" />
+    <geometry>
+      <cylinder radius="0.06" length="0.04" />
+    </geometry>
+    <material name="wheel_material">
+        <color rgba="${wheel_color}"/>
+    </material>
+  </visual>
 </link>
+<gazebo reference="${prefix}_wheel">
+  <material>Gazebo/Black</material>
+</gazebo>
 </xacro:macro>
 <xacro:macro name="wheel_joint" params="prefix origin">
