Commit message: Outdoor Navigation

File: robot_description/urdf/robot_base.xacro (robot description, xacro)
@@ -41,6 +41,6 @@
  <joint name="base_footprint_joint" type="fixed">
     <origin xyz="0 0 -0.06" rpy="0 0 0" />
-    <parent link="base_link" />
-    <child link="base_footprint" />
+    <parent link="base_footprint" />
+    <child link="base_link" />
  </joint>
   <link name="base_footprint">

File: robot_description/urdf/robot_essentials.xacro (robot description, xacro)
@@ -20,4 +20,5 @@
     <geometry>
       <cylinder radius="0.06" length="0.04" />
+      <!--mesh filename="package://robot_description/meshes/wheel.dae"/-->
     </geometry>
     <material name="wheel_material">

Commit message: Problems in the indoor navigation fixed

File: robot_description/urdf/robot_base.xacro (robot description, xacro)
@@ -40,5 +40,5 @@
   <!-- Base FootPrint Link-->
  <joint name="base_footprint_joint" type="fixed">
-    <origin xyz="0 0 -0.06" rpy="0 0 0" />
+    <origin xyz="0 0 0.06" rpy="0 0 0" />
     <parent link="base_footprint" />
     <child link="base_link" />
